File: kicad/i2s-amp-shim.kicad_pcb (KiCad board)
At the start: 2 copper layers, 17.5 x 24.9 mm, 2 parts, among them J1 Feather 3V-A2, J2 MAX98357 #3006

Commit message: Flat SMT socket models and render-only Feather + amp
Sockets now use flat-SMT right-angle models (make_3d.py, FreeCAD) instead
of KiCad's through-hole part. Add board-only, render-only footprints that
show an Adafruit Feather RP2350 and the MAX98357 (#3006) plugged into J1
and J2, using Adafruit_CAD_Parts models plus KiCad male headers. No copper
or schematic change. Ignore KiCad plot outputs and local history.

Co-Authored-By: Claude Opus 5.5 (1M context) <noreply@anthropic.com>
Parts:
- added VIS1: Render_Feather_RP2350_on_J1, i2s-amp-shim:Render_Feather_RP2350_on_J1, F.Cu at (-1.70, 16.4)
- added VIS2: Render_MAX98357_on_J2, i2s-amp-shim:Render_MAX98357_on_J2, F.Cu at (18.0, 11.3)
